File: kicad/tkl_low_profile.kicad_pcb (KiCad board)
At the start: 2 copper layers, 0 parts

Commit message: wip
Parts:
- added C1: 0.1u, ScottoKeebs_Components:Capacitor_0603, B.Cu at (172.0, 64.0)
- added D1: D, ScottoKeebs_Components:Diode_SOD-123, F.Cu at (20.0, 27.0)
- added D10: D, ScottoKeebs_Components:Diode_SOD-123, F.Cu at (229.6, 27.0)
- added D11: D, ScottoKeebs_Components:Diode_SOD-123, F.Cu at (248.6, 27.0)
- added D12: D, ScottoKeebs_Components:Diode_SOD-123, F.Cu at (267.6, 27.0)
- added D13: D, ScottoKeebs_Components:Diode_SOD-123, F.Cu at (286.7, 27.0)
- added D14: D, ScottoKeebs_Components:Diode_SOD-123, F.Cu at (315.3, 27.0)
- added D15: D, ScottoKeebs_Components:Diode_SOD-123, F.Cu at (334.3, 27.0)
- added D16: D, ScottoKeebs_Components:Diode_SOD-123, F.Cu at (353.4, 27.0)
- added D17: D, ScottoKeebs_Components:Diode_SOD-123, F.Cu at (20.0, 50.8)
- added D18: D, ScottoKeebs_Components:Diode_SOD-123, F.Cu at (39.0, 50.8)
- added D19: D, ScottoKeebs_Components:Diode_SOD-123, F.Cu at (58.1, 50.8)
- added D2: D, ScottoKeebs_Components:Diode_SOD-123, F.Cu at (51.8, 27.0)
- added D20: D, ScottoKeebs_Components:Diode_SOD-123, F.Cu at (77.2, 50.8)
- added D21: D, ScottoKeebs_Components:Diode_SOD-123, F.Cu at (96.2, 50.8)
- added D22: D, ScottoKeebs_Components:Diode_SOD-123, F.Cu at (115.2, 50.8)
- added D23: D, ScottoKeebs_Components:Diode_SOD-123, F.Cu at (134.3, 50.8)
- added D24: D, ScottoKeebs_Components:Diode_SOD-123, F.Cu at (153.3, 50.8)
- added D25: D, ScottoKeebs_Components:Diode_SOD-123, F.Cu at (172.4, 50.8)
- added D26: D, ScottoKeebs_Components:Diode_SOD-123, F.Cu at (191.4, 50.8)
- added D27: D, ScottoKeebs_Components:Diode_SOD-123, F.Cu at (210.5, 50.8)
- added D28: D, ScottoKeebs_Components:Diode_SOD-123, F.Cu at (229.6, 50.8)
- added D29: D, ScottoKeebs_Components:Diode_SOD-123, F.Cu at (248.6, 50.8)
- added D3: D, ScottoKeebs_Components:Diode_SOD-123, F.Cu at (70.8, 27.0)
- added D30: D, ScottoKeebs_Components:Diode_SOD-123, F.Cu at (277.2, 50.8)
- added D31: D, ScottoKeebs_Components:Diode_SOD-123, F.Cu at (315.3, 50.8)
- added D32: D, ScottoKeebs_Components:Diode_SOD-123, F.Cu at (334.3, 50.8)
- added D33: D, ScottoKeebs_Components:Diode_SOD-123, F.Cu at (353.4, 50.8)
- added D34: D, ScottoKeebs_Components:Diode_SOD-123, F.Cu at (24.8, 69.9)
- added D35: D, ScottoKeebs_Components:Diode_SOD-123, F.Cu at (48.6, 69.9)
- added D36: D, ScottoKeebs_Components:Diode_SOD-123, F.Cu at (67.6, 69.9)
- added D37: D, ScottoKeebs_Components:Diode_SOD-123, F.Cu at (86.7, 69.9)
- added D38: D, ScottoKeebs_Components:Diode_SOD-123, F.Cu at (105.7, 69.9)
- added D39: D, ScottoKeebs_Components:Diode_SOD-123, F.Cu at (124.8, 69.9)
- added D4: D, ScottoKeebs_Components:Diode_SOD-123, F.Cu at (89.9, 27.0)
- added D40: D, ScottoKeebs_Components:Diode_SOD-123, F.Cu at (143.8, 69.9)
- added D41: D, ScottoKeebs_Components:Diode_SOD-123, F.Cu at (162.9, 69.9)
- added D42: D, ScottoKeebs_Components:Diode_SOD-123, F.Cu at (181.9, 69.9)
- added D43: D, ScottoKeebs_Components:Diode_SOD-123, F.Cu at (201.0, 69.9)
- added D44: D, ScottoKeebs_Components:Diode_SOD-123, F.Cu at (220.0, 69.9)
- added D45: D, ScottoKeebs_Components:Diode_SOD-123, F.Cu at (239.1, 69.9)
- added D46: D, ScottoKeebs_Components:Diode_SOD-123, F.Cu at (258.1, 69.9)
- added D47: D, ScottoKeebs_Components:Diode_SOD-123, F.Cu at (281.9, 69.9)
- added D48: D, ScottoKeebs_Components:Diode_SOD-123, F.Cu at (315.3, 69.9)
- added D49: D, ScottoKeebs_Components:Diode_SOD-123, F.Cu at (334.3, 69.9)
- added D5: D, ScottoKeebs_Components:Diode_SOD-123, F.Cu at (108.9, 27.0)
- added D50: D, ScottoKeebs_Components:Diode_SOD-123, F.Cu at (353.4, 69.9)
- added D51: D, ScottoKeebs_Components:Diode_SOD-123, F.Cu at (27.1, 88.9)
- added D52: D, ScottoKeebs_Components:Diode_SOD-123, F.Cu at (53.3, 88.9)
- added D53: D, ScottoKeebs_Components:Diode_SOD-123, F.Cu at (72.4, 88.9)
- added D54: D, ScottoKeebs_Components:Diode_SOD-123, F.Cu at (91.4, 88.9)
- added D55: D, ScottoKeebs_Components:Diode_SOD-123, F.Cu at (110.5, 88.9)
- added D56: D, ScottoKeebs_Components:Diode_SOD-123, F.Cu at (129.5, 88.9)
- added D57: D, ScottoKeebs_Components:Diode_SOD-123, F.Cu at (148.6, 88.9)
- added D58: D, ScottoKeebs_Components:Diode_SOD-123, F.Cu at (167.6, 88.9)
- added D59: D, ScottoKeebs_Components:Diode_SOD-123, F.Cu at (186.7, 88.9)
- added D6: D, ScottoKeebs_Components:Diode_SOD-123, F.Cu at (140.6, 27.0)
- added D60: D, ScottoKeebs_Components:Diode_SOD-123, F.Cu at (205.7, 88.9)
- added D61: D, ScottoKeebs_Components:Diode_SOD-123, F.Cu at (224.8, 88.9)
- added D62: D, ScottoKeebs_Components:Diode_SOD-123, F.Cu at (243.8, 88.9)
- added D63: D, ScottoKeebs_Components:Diode_SOD-123, F.Cu at (274.8, 88.9)
- added D64: D, ScottoKeebs_Components:Diode_SOD-123, F.Cu at (31.9, 108.0)
- added D65: D, ScottoKeebs_Components:Diode_SOD-123, F.Cu at (62.9, 108.0)
- added D66: D, ScottoKeebs_Components:Diode_SOD-123, F.Cu at (81.9, 108.0)
- added D67: D, ScottoKeebs_Components:Diode_SOD-123, F.Cu at (101.0, 108.0)
- added D68: D, ScottoKeebs_Components:Diode_SOD-123, F.Cu at (120.0, 108.0)
- added D69: D, ScottoKeebs_Components:Diode_SOD-123, F.Cu at (139.1, 108.0)
- added D7: D, ScottoKeebs_Components:Diode_SOD-123, F.Cu at (159.7, 27.0)
- added D70: D, ScottoKeebs_Components:Diode_SOD-123, F.Cu at (158.1, 108.0)
- added D71: D, ScottoKeebs_Components:Diode_SOD-123, F.Cu at (177.2, 108.0)
- added D72: D, ScottoKeebs_Components:Diode_SOD-123, F.Cu at (196.2, 108.0)
- added D73: D, ScottoKeebs_Components:Diode_SOD-123, F.Cu at (215.3, 108.0)
- added D74: D, ScottoKeebs_Components:Diode_SOD-123, F.Cu at (234.3, 108.0)
- added D75: D, ScottoKeebs_Components:Diode_SOD-123, F.Cu at (270.0, 108.0)
- added D76: D, ScottoKeebs_Components:Diode_SOD-123, F.Cu at (334.3, 108.0)
- added D77: D, ScottoKeebs_Components:Diode_SOD-123, F.Cu at (22.4, 127.0)
- added D78: D, ScottoKeebs_Components:Diode_SOD-123, F.Cu at (46.2, 127.0)
- added D79: D, ScottoKeebs_Components:Diode_SOD-123, F.Cu at (70.0, 127.0)
- added D8: D, ScottoKeebs_Components:Diode_SOD-123, F.Cu at (178.7, 27.0)
- added D80: D, ScottoKeebs_Components:Diode_SOD-123, F.Cu at (141.4, 127.0)
- added D81: D, ScottoKeebs_Components:Diode_SOD-123, F.Cu at (212.9, 127.0)
- added D82: D, ScottoKeebs_Components:Diode_SOD-123, F.Cu at (236.7, 127.0)
- added D83: D, ScottoKeebs_Components:Diode_SOD-123, F.Cu at (260.5, 127.0)
- added D84: D, ScottoKeebs_Components:Diode_SOD-123, F.Cu at (284.3, 127.0)
- added D85: D, ScottoKeebs_Components:Diode_SOD-123, F.Cu at (315.3, 127.0)
- added D86: D, ScottoKeebs_Components:Diode_SOD-123, F.Cu at (334.3, 127.0)
- added D87: D, ScottoKeebs_Components:Diode_SOD-123, F.Cu at (353.4, 127.0)
- added D9: D, ScottoKeebs_Components:Diode_SOD-123, F.Cu at (197.8, 27.0)
- added JBAT1: JST-PH, ScottoKeebs_Components:Connector_1x02_JST-PH, B.Cu at (210.0, 80.0)
- added JLED1: LED_HARNESS, Connector_Wire:SolderWire-0.25sqmm_1x02_P4.2mm_D0.65mm_OD1.7mm_Relief, B.Cu at (340.0, 12.0)
- added Q1: NMOS, Package_TO_SOT_SMD:SOT-23, B.Cu at (210.0, 48.0)
- added R1: 4.7k, ScottoKeebs_Components:Resistor_0805, B.Cu at (172.0, 52.0)
- added R2: 4.7k, ScottoKeebs_Components:Resistor_0805, B.Cu at (172.0, 56.0)
- added R3: 10k, ScottoKeebs_Components:Resistor_0805, B.Cu at (172.0, 60.0)
- added R4: 100, ScottoKeebs_Components:Resistor_0805, B.Cu at (210.0, 54.0)
- added R5: 100k, ScottoKeebs_Components:Resistor_0805, B.Cu at (210.0, 58.0)
- added SW1: SW_Push, MX_V2_Kailh_PG1353_Hotswap:Kailh-PG1353-Hotswap-1U, B.Cu at (20.0, 20.0)
- added SW10: SW_Push, MX_V2_Kailh_PG1353_Hotswap:Kailh-PG1353-Hotswap-1U, B.Cu at (229.6, 20.0)
- added SW11: SW_Push, MX_V2_Kailh_PG1353_Hotswap:Kailh-PG1353-Hotswap-1U, B.Cu at (248.6, 20.0)
- added SW12: SW_Push, MX_V2_Kailh_PG1353_Hotswap:Kailh-PG1353-Hotswap-1U, B.Cu at (267.6, 20.0)
- added SW13: SW_Push, MX_V2_Kailh_PG1353_Hotswap:Kailh-PG1353-Hotswap-1U, B.Cu at (286.7, 20.0)
- added SW14: SW_Push, MX_V2_Kailh_PG1353_Hotswap:Kailh-PG1353-Hotswap-1U, B.Cu at (315.3, 20.0)
- added SW15: SW_Push, MX_V2_Kailh_PG1353_Hotswap:Kailh-PG1353-Hotswap-1U, B.Cu at (334.3, 20.0)
- added SW16: SW_Push, MX_V2_Kailh_PG1353_Hotswap:Kailh-PG1353-Hotswap-1U, B.Cu at (353.4, 20.0)
- added SW17: SW_Push, MX_V2_Kailh_PG1353_Hotswap:Kailh-PG1353-Hotswap-1U, B.Cu at (20.0, 43.8)
- added SW18: SW_Push, MX_V2_Kailh_PG1353_Hotswap:Kailh-PG1353-Hotswap-1U, B.Cu at (39.0, 43.8)
- added SW19: SW_Push, MX_V2_Kailh_PG1353_Hotswap:Kailh-PG1353-Hotswap-1U, B.Cu at (58.1, 43.8)
- added SW2: SW_Push, MX_V2_Kailh_PG1353_Hotswap:Kailh-PG1353-Hotswap-1U, B.Cu at (51.8, 20.0)
- added SW20: SW_Push, MX_V2_Kailh_PG1353_Hotswap:Kailh-PG1353-Hotswap-1U, B.Cu at (77.2, 43.8)
- added SW21: SW_Push, MX_V2_Kailh_PG1353_Hotswap:Kailh-PG1353-Hotswap-1U, B.Cu at (96.2, 43.8)
- added SW22: SW_Push, MX_V2_Kailh_PG1353_Hotswap:Kailh-PG1353-Hotswap-1U, B.Cu at (115.2, 43.8)
- added SW23: SW_Push, MX_V2_Kailh_PG1353_Hotswap:Kailh-PG1353-Hotswap-1U, B.Cu at (134.3, 43.8)
- added SW24: SW_Push, MX_V2_Kailh_PG1353_Hotswap:Kailh-PG1353-Hotswap-1U, B.Cu at (153.3, 43.8)
- added SW25: SW_Push, MX_V2_Kailh_PG1353_Hotswap:Kailh-PG1353-Hotswap-1U, B.Cu at (172.4, 43.8)
- added SW26: SW_Push, MX_V2_Kailh_PG1353_Hotswap:Kailh-PG1353-Hotswap-1U, B.Cu at (191.4, 43.8)
- added SW27: SW_Push, MX_V2_Kailh_PG1353_Hotswap:Kailh-PG1353-Hotswap-1U, B.Cu at (210.5, 43.8)
- added SW28: SW_Push, MX_V2_Kailh_PG1353_Hotswap:Kailh-PG1353-Hotswap-1U, B.Cu at (229.6, 43.8)
- added SW29: SW_Push, MX_V2_Kailh_PG1353_Hotswap:Kailh-PG1353-Hotswap-1U, B.Cu at (248.6, 43.8)
- added SW3: SW_Push, MX_V2_Kailh_PG1353_Hotswap:Kailh-PG1353-Hotswap-1U, B.Cu at (70.8, 20.0)
- added SW30: SW_Push, MX_V2_Kailh_PG1353_Hotswap:Kailh-PG1353-Hotswap-2U, B.Cu at (277.2, 43.8)
- added SW31: SW_Push, MX_V2_Kailh_PG1353_Hotswap:Kailh-PG1353-Hotswap-1U, B.Cu at (315.3, 43.8)
- added SW32: SW_Push, MX_V2_Kailh_PG1353_Hotswap:Kailh-PG1353-Hotswap-1U, B.Cu at (334.3, 43.8)
- added SW33: SW_Push, MX_V2_Kailh_PG1353_Hotswap:Kailh-PG1353-Hotswap-1U, B.Cu at (353.4, 43.8)
- added SW34: SW_Push, MX_V2_Kailh_PG1353_Hotswap:Kailh-PG1353-Hotswap-1.5U, B.Cu at (24.8, 62.9)
- added SW35: SW_Push, MX_V2_Kailh_PG1353_Hotswap:Kailh-PG1353-Hotswap-1U, B.Cu at (48.6, 62.9)
- added SW36: SW_Push, MX_V2_Kailh_PG1353_Hotswap:Kailh-PG1353-Hotswap-1U, B.Cu at (67.6, 62.9)
- added SW37: SW_Push, MX_V2_Kailh_PG1353_Hotswap:Kailh-PG1353-Hotswap-1U, B.Cu at (86.7, 62.9)
- added SW38: SW_Push, MX_V2_Kailh_PG1353_Hotswap:Kailh-PG1353-Hotswap-1U, B.Cu at (105.7, 62.9)
- added SW39: SW_Push, MX_V2_Kailh_PG1353_Hotswap:Kailh-PG1353-Hotswap-1U, B.Cu at (124.8, 62.9)
- added SW4: SW_Push, MX_V2_Kailh_PG1353_Hotswap:Kailh-PG1353-Hotswap-1U, B.Cu at (89.9, 20.0)
- added SW40: SW_Push, MX_V2_Kailh_PG1353_Hotswap:Kailh-PG1353-Hotswap-1U, B.Cu at (143.8, 62.9)
- added SW41: SW_Push, MX_V2_Kailh_PG1353_Hotswap:Kailh-PG1353-Hotswap-1U, B.Cu at (162.9, 62.9)
- added SW42: SW_Push, MX_V2_Kailh_PG1353_Hotswap:Kailh-PG1353-Hotswap-1U, B.Cu at (181.9, 62.9)
- added SW43: SW_Push, MX_V2_Kailh_PG1353_Hotswap:Kailh-PG1353-Hotswap-1U, B.Cu at (201.0, 62.9)
- added SW44: SW_Push, MX_V2_Kailh_PG1353_Hotswap:Kailh-PG1353-Hotswap-1U, B.Cu at (220.0, 62.9)
- added SW45: SW_Push, MX_V2_Kailh_PG1353_Hotswap:Kailh-PG1353-Hotswap-1U, B.Cu at (239.1, 62.9)
- added SW46: SW_Push, MX_V2_Kailh_PG1353_Hotswap:Kailh-PG1353-Hotswap-1U, B.Cu at (258.1, 62.9)
- added SW47: SW_Push, MX_V2_Kailh_PG1353_Hotswap:Kailh-PG1353-Hotswap-1.5U, B.Cu at (281.9, 62.9)
- added SW48: SW_Push, MX_V2_Kailh_PG1353_Hotswap:Kailh-PG1353-Hotswap-1U, B.Cu at (315.3, 62.9)
- added SW49: SW_Push, MX_V2_Kailh_PG1353_Hotswap:Kailh-PG1353-Hotswap-1U, B.Cu at (334.3, 62.9)
- added SW5: SW_Push, MX_V2_Kailh_PG1353_Hotswap:Kailh-PG1353-Hotswap-1U, B.Cu at (108.9, 20.0)
- added SW50: SW_Push, MX_V2_Kailh_PG1353_Hotswap:Kailh-PG1353-Hotswap-1U, B.Cu at (353.4, 62.9)
- added SW51: SW_Push, MX_V2_Kailh_PG1353_Hotswap:Kailh-PG1353-Hotswap-1.75U, B.Cu at (27.1, 81.9)
- added SW52: SW_Push, MX_V2_Kailh_PG1353_Hotswap:Kailh-PG1353-Hotswap-1U, B.Cu at (53.3, 81.9)
- added SW53: SW_Push, MX_V2_Kailh_PG1353_Hotswap:Kailh-PG1353-Hotswap-1U, B.Cu at (72.4, 81.9)
- added SW54: SW_Push, MX_V2_Kailh_PG1353_Hotswap:Kailh-PG1353-Hotswap-1U, B.Cu at (91.4, 81.9)
- added SW55: SW_Push, MX_V2_Kailh_PG1353_Hotswap:Kailh-PG1353-Hotswap-1U, B.Cu at (110.5, 81.9)
- added SW56: SW_Push, MX_V2_Kailh_PG1353_Hotswap:Kailh-PG1353-Hotswap-1U, B.Cu at (129.5, 81.9)
- added SW57: SW_Push, MX_V2_Kailh_PG1353_Hotswap:Kailh-PG1353-Hotswap-1U, B.Cu at (148.6, 81.9)
- added SW58: SW_Push, MX_V2_Kailh_PG1353_Hotswap:Kailh-PG1353-Hotswap-1U, B.Cu at (167.6, 81.9)
- added SW59: SW_Push, MX_V2_Kailh_PG1353_Hotswap:Kailh-PG1353-Hotswap-1U, B.Cu at (186.7, 81.9)
- added SW6: SW_Push, MX_V2_Kailh_PG1353_Hotswap:Kailh-PG1353-Hotswap-1U, B.Cu at (140.6, 20.0)
- added SW60: SW_Push, MX_V2_Kailh_PG1353_Hotswap:Kailh-PG1353-Hotswap-1U, B.Cu at (205.7, 81.9)
- added SW61: SW_Push, MX_V2_Kailh_PG1353_Hotswap:Kailh-PG1353-Hotswap-1U, B.Cu at (224.8, 81.9)
- added SW62: SW_Push, MX_V2_Kailh_PG1353_Hotswap:Kailh-PG1353-Hotswap-1U, B.Cu at (243.8, 81.9)
- added SW63: SW_Push, MX_V2_Kailh_PG1353_Hotswap:Kailh-PG1353-Hotswap-2.25U, B.Cu at (274.8, 81.9)
- added SW64: SW_Push, MX_V2_Kailh_PG1353_Hotswap:Kailh-PG1353-Hotswap-2.25U, B.Cu at (31.9, 101.0)
- added SW65: SW_Push, MX_V2_Kailh_PG1353_Hotswap:Kailh-PG1353-Hotswap-1U, B.Cu at (62.9, 101.0)
- added SW66: SW_Push, MX_V2_Kailh_PG1353_Hotswap:Kailh-PG1353-Hotswap-1U, B.Cu at (81.9, 101.0)
- added SW67: SW_Push, MX_V2_Kailh_PG1353_Hotswap:Kailh-PG1353-Hotswap-1U, B.Cu at (101.0, 101.0)
- added SW68: SW_Push, MX_V2_Kailh_PG1353_Hotswap:Kailh-PG1353-Hotswap-1U, B.Cu at (120.0, 101.0)
- added SW69: SW_Push, MX_V2_Kailh_PG1353_Hotswap:Kailh-PG1353-Hotswap-1U, B.Cu at (139.1, 101.0)
- added SW7: SW_Push, MX_V2_Kailh_PG1353_Hotswap:Kailh-PG1353-Hotswap-1U, B.Cu at (159.7, 20.0)
- added SW70: SW_Push, MX_V2_Kailh_PG1353_Hotswap:Kailh-PG1353-Hotswap-1U, B.Cu at (158.1, 101.0)
- added SW71: SW_Push, MX_V2_Kailh_PG1353_Hotswap:Kailh-PG1353-Hotswap-1U, B.Cu at (177.2, 101.0)
- added SW72: SW_Push, MX_V2_Kailh_PG1353_Hotswap:Kailh-PG1353-Hotswap-1U, B.Cu at (196.2, 101.0)
- added SW73: SW_Push, MX_V2_Kailh_PG1353_Hotswap:Kailh-PG1353-Hotswap-1U, B.Cu at (215.3, 101.0)
- added SW74: SW_Push, MX_V2_Kailh_PG1353_Hotswap:Kailh-PG1353-Hotswap-1U, B.Cu at (234.3, 101.0)
- added SW75: SW_Push, MX_V2_Kailh_PG1353_Hotswap:Kailh-PG1353-Hotswap-2.75U, B.Cu at (270.0, 101.0)
- added SW76: SW_Push, MX_V2_Kailh_PG1353_Hotswap:Kailh-PG1353-Hotswap-1U, B.Cu at (334.3, 101.0)
- added SW77: SW_Push, MX_V2_Kailh_PG1353_Hotswap:Kailh-PG1353-Hotswap-1.25U, B.Cu at (22.4, 120.0)
- added SW78: SW_Push, MX_V2_Kailh_PG1353_Hotswap:Kailh-PG1353-Hotswap-1.25U, B.Cu at (46.2, 120.0)
- added SW79: SW_Push, MX_V2_Kailh_PG1353_Hotswap:Kailh-PG1353-Hotswap-1.25U, B.Cu at (70.0, 120.0)
- added SW8: SW_Push, MX_V2_Kailh_PG1353_Hotswap:Kailh-PG1353-Hotswap-1U, B.Cu at (178.7, 20.0)
- added SW80: SW_Push, MX_V2_Kailh_PG1353_Hotswap:Kailh-PG1353-Hotswap-6.25U, B.Cu at (141.4, 120.0)
- added SW81: SW_Push, MX_V2_Kailh_PG1353_Hotswap:Kailh-PG1353-Hotswap-1.25U, B.Cu at (212.9, 120.0)
- added SW82: SW_Push, MX_V2_Kailh_PG1353_Hotswap:Kailh-PG1353-Hotswap-1.25U, B.Cu at (236.7, 120.0)
- added SW83: SW_Push, MX_V2_Kailh_PG1353_Hotswap:Kailh-PG1353-Hotswap-1.25U, B.Cu at (260.5, 120.0)
- added SW84: SW_Push, MX_V2_Kailh_PG1353_Hotswap:Kailh-PG1353-Hotswap-1.25U, B.Cu at (284.3, 120.0)
- added SW85: SW_Push, MX_V2_Kailh_PG1353_Hotswap:Kailh-PG1353-Hotswap-1U, B.Cu at (315.3, 120.0)
- added SW86: SW_Push, MX_V2_Kailh_PG1353_Hotswap:Kailh-PG1353-Hotswap-1U, B.Cu at (334.3, 120.0)
- added SW87: SW_Push, MX_V2_Kailh_PG1353_Hotswap:Kailh-PG1353-Hotswap-1U, B.Cu at (353.4, 120.0)
- added SW9: SW_Push, MX_V2_Kailh_PG1353_Hotswap:Kailh-PG1353-Hotswap-1U, B.Cu at (197.8, 20.0)
- added SWPWR1: Power_Switch, ScottoKeebs_Components:Switch_MSK12C02, B.Cu at (320.0, 11.4)
- added U1: Nice_Nano_V2, ScottoKeebs_MCU:Nice_Nano_V2, B.Cu at (186.7, 26.3)
- added U2: MCP23017, Package_SO:SOIC-28W_7.5x17.9mm_P1.27mm, B.Cu at (186.7, 60.0)
Routing:
- net COL2: track 0.00 -> 860.4 mm
- net COL1: track 0.00 -> 830.6 mm
- net COL0: track 0.00 -> 825.8 mm
- net COL5: track 0.00 -> 743.6 mm
- net COL3: track 0.00 -> 693.2 mm
- net COL4: track 0.00 -> 682.5 mm
- net COL6: track 0.00 -> 512.9 mm
- net COL7: track 0.00 -> 466.0 mm
- net COL8: track 0.00 -> 450.7 mm
- net ROW5: track 0.00 -> 441.1 mm
- net ROW3: track 0.00 -> 431.6 mm
- net COL10: track 0.00 -> 401.0 mm
- net COL9: track 0.00 -> 393.0 mm
- net ROW2: track 0.00 -> 381.4 mm
- net ROW0: track 0.00 -> 337.1 mm
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Other:
- board outline added: 356.4 x 123.1 mm
